File: pcb/binary_clock.sch (EAGLE design)
At the start: 24 parts

Commit message: More 100nFs added, short circuit corrected, text added
Parts:
- added C2, C3, C4, C5: (no value), rcl:C-EUC0603K
Connections:
- net +5V: now also C2.1, C3.1, C4.1, C5.1
- net GND: now also C2.2, C3.2, C4.2, C5.2
Changed lines of the file:
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@@
 <part name="OSC" library="SparkFun-Clocks" deviceset="OSCILLATOR" device="SMD-5X3"/>
 <part name="R3" library="rcl" deviceset="R-EU_" device="R1206"/>
+<part name="C2" library="rcl" deviceset="C-EU" device="C0603K"/>
+<part name="C3" library="rcl" deviceset="C-EU" device="C0603K"/>
+<part name="C4" library="rcl" deviceset="C-EU" device="C0603K"/>
+<part name="C5" library="rcl" deviceset="C-EU" device="C0603K"/>
 </parts>
 <sheets>
@@
 <instance part="OSC" gate="G$1" x="-30.48" y="96.52"/>
 <instance part="R3" gate="G$1" x="12.7" y="60.96"/>
+<instance part="C2" gate="G$1" x="-48.26" y="40.64"/>
+<instance part="C3" gate="G$1" x="-43.18" y="40.64"/>
+<instance part="C4" gate="G$1" x="-38.1" y="40.64"/>
+<instance part="C5" gate="G$1" x="-33.02" y="40.64"/>
 </instances>
 <busses>
@@
 <wire x1="-53.34" y1="35.56" x2="-53.34" y2="33.02" width="0.1524" layer="91"/>
 <label x="-53.34" y="33.02" size="0.8128" layer="95" rot="R180" xref="yes"/>
+<pinref part="C2" gate="G$1" pin="2"/>
+<wire x1="-53.34" y1="35.56" x2="-48.26" y2="35.56" width="0.1524" layer="91"/>
+<pinref part="C3" gate="G$1" pin="2"/>
+<wire x1="-48.26" y1="35.56" x2="-43.18" y2="35.56" width="0.1524" layer="91"/>
+<pinref part="C4" gate="G$1" pin="2"/>
+<wire x1="-43.18" y1="35.56" x2="-38.1" y2="35.56" width="0.1524" layer="91"/>
+<pinref part="C5" gate="G$1" pin="2"/>
+<wire x1="-38.1" y1="35.56" x2="-33.02" y2="35.56" width="0.1524" layer="91"/>
 </segment>
 <segment>
@@
 <wire x1="-53.34" y1="43.18" x2="-53.34" y2="45.72" width="0.1524" layer="91"/>
 <label x="-53.34" y="45.72" size="0.8128" layer="95" rot="R180" xref="yes"/>
-</segment>
-<segment>
+<pinref part="C2" gate="G$1" pin="1"/>
+<wire x1="-53.34" y1="43.18" x2="-48.26" y2="43.18" width="0.1524" layer="91"/>
+<pinref part="C3" gate="G$1" pin="1"/>
+<wire x1="-48.26" y1="43.18" x2="-43.18" y2="43.18" width="0.1524" layer="91"/>
+<pinref part="C4" gate="G$1" pin="1"/>
+<wire x1="-43.18" y1="43.18" x2="-38.1" y2="43.18" width="0.1524" layer="91"/>
+<pinref part="C5" gate="G$1" pin="1"/>
+<wire x1="-38.1" y1="43.18" x2="-33.02" y2="43.18" width="0.1524" layer="91"/>
+</segment>
+<segment>
