File: panelized/binary_clock_panelized.brd (EAGLE design)
At the start: 163 x 100 mm, 244 parts

Commit message: Panelized version corrected
Parts:
- removed C31, C32, C33, C34, C35: (no value), rcl:C0603K
- removed LED103, LED104, LED105, LED106, LED107, LED108, LED109, LED110, LED111, LED112, LED113, LED114, LED115, LED116, LED117, LED118, LED119: APA102-5050, SparkFun-LED:APA102-5050
- removed MCU: TINY25-20SU, avr-4:SOIC8
- removed OSC: OSCILLATORSMD-5X3, SparkFun-Clocks:OSCILLATOR-SMD-5X3.2
- removed R19, R20, R21: (no value), rcl:R1206
- removed SET: SET, SparkFun-Switches:TACTILE_SWITCH_SMD_5.2MM
- moved LED4 144.0 mm to (6.47, 58.2)
- moved LED5 144.0 mm to (14.1, 58.2)
- moved LED17 140.4 mm to (21.7, 65.9), turned to 90 degrees
- moved LED3 137.4 mm to (6.47, 65.9), turned to 90 degrees
- moved LED6 137.4 mm to (21.7, 58.2), turned to 270 degrees
- moved LED16 125.7 mm to (29.3, 65.9), turned to 90 degrees
- moved LED7 122.3 mm to (29.3, 58.2), turned to 270 degrees
- moved LED2 122.3 mm to (14.1, 65.9), turned to 90 degrees
- moved C3 116.4 mm to (37.0, 57.1)
- moved C5 116.4 mm to (37.0, 68.6)
- moved C1 116.4 mm to (9.33, 64.9)
- moved C2 116.4 mm to (14.1, 57.1)
- moved C4 116.4 mm to (21.7, 71.7)
- moved LED1 116.4 mm to (14.1, 73.5)
- moved R1 116.4 mm to (10.3, 69.7)
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Connections:
- removed net +5V: C1.1, C2.1, C3.1, C4.1, C5.1, LED1.P4, LED10.P4, LED11.P4, LED12.P4, LED13.P4, LED14.P4, LED15.P4, LED16.P4, LED2.P4, LED3.P4, LED4.P4, LED5.P4, LED6.P4, LED7.P4, LED8.P4, LED9.P4, MCU.8, OSC.4
- removed net GND: C1.2, C2.2, C3.2, C4.2, C5.2, LED1.P3, LED10.P3, LED11.P3, LED12.P3, LED13.P3, LED14.P3, LED15.P3, LED16.P3, LED17.P3, LED2.P3, LED3.P3, LED4.P3, LED5.P3, LED6.P3, LED7.P3, LED8.P3, LED9.P3, MCU.4, OSC.2, SET.3, SET.4
- removed net LED_CK: MCU.6, R1.1
- removed net LED_D: MCU.5, R2.1
- removed net N$11 (its old number): LED10.P1, LED9.P6
- removed net N$12 (its old number): LED10.P2, LED9.P5
- removed net N$247: LED103.P5, LED112.P2
- removed net N$248: LED103.P6, LED112.P1
- removed net N$249: LED112.P5, LED113.P2
- removed net N$250: LED112.P6, LED113.P1
- removed net N$251: LED113.P5, LED114.P2
- removed net N$252: LED113.P6, LED114.P1
- removed net N$253: LED114.P5, LED115.P2
- removed net N$254: LED114.P6, LED115.P1
- removed net N$255: LED106.P5, LED107.P2
- removed net N$256: LED106.P6, LED107.P1
- removed net N$257: LED107.P5, LED108.P2
- removed net N$258: LED107.P6, LED108.P1
- removed net N$259: LED108.P5, LED109.P2
- removed net N$260: LED108.P6, LED109.P1
- removed net N$261: LED109.P5, LED110.P2
- removed net N$262: LED109.P6, LED110.P1
- removed net N$263: LED110.P5, LED111.P2
- removed net N$264: LED110.P6, LED111.P1
- removed net N$265: LED111.P4
- removed net N$266: LED104.P5, LED105.P2
- removed net N$267: LED104.P6, LED105.P1
- removed net N$268: LED104.P1, LED119.P6
- removed net N$269: LED104.P2, LED119.P5
- removed net N$270: LED118.P6, LED119.P1
- removed net N$271: LED118.P5, LED119.P2
- removed net N$272: LED117.P6, LED118.P1
- removed net N$273: LED117.P5, LED118.P2
- removed net N$274: LED116.P6, LED117.P1
- removed net N$275: LED116.P5, LED117.P2
- removed net N$276: LED105.P6, LED106.P1
- removed net N$277: LED105.P5, LED106.P2
- removed net N$278: LED111.P6
- removed net N$279: LED111.P5
- removed net N$280: LED115.P6, LED116.P1
- removed net N$281: LED103.P1, R20.2
- removed net N$282: LED103.P2, R19.2
- removed net N$283: LED115.P5, LED116.P2
- removed net N$287: R21.2, SET6.1, SET6.2
- removed net N$31 (its old number): LED17.P6
- removed net N$34 (its old number): LED17.P5
- removed net N$35 (its old number): MCU.2, OSC.3
- removed net N$36 (its old number): R3.2, SET.1, SET.2
- removed net N$63 (its old number): LED17.P4
- removed net SW: MCU.7, R3.1
- new net N$19: LED9.P4
- new net N$22: LED17.P6, LED2.P1
- new net N$23: LED17.P5, LED2.P2
- new net N$41: R3.2, SET1.1, SET1.2
- net +5V1: now also C1.1, C2.1, C3.1, C4.1, C5.1, LED1.P4, LED10.P4, LED11.P4, LED12.P4, LED13.P4, LED14.P4, LED15.P4, LED16.P4, LED17.P4, LED2.P4, LED3.P4, LED4.P4, LED5.P4, LED6.P4, LED7.P4, LED8.P4; no longer C10.1, C6.1, C7.1, C8.1, C9.1, LED18.P4, LED19.P4, LED20.P4, LED21.P4, LED22.P4, LED23.P4, LED24.P4, LED25.P4, LED27.P4, LED28.P4, LED29.P4, LED30.P4, LED31.P4, LED32.P4, LED33.P4, LED34.P4
- net +5V2: now also C10.1, C6.1, C7.1, C8.1, C9.1, LED18.P4, LED19.P4, LED20.P4, LED21.P4, LED22.P4, LED23.P4, LED24.P4, LED25.P4, LED27.P4, LED28.P4, LED29.P4, LED30.P4, LED31.P4, LED32.P4, LED33.P4, LED34.P4; no longer C11.1, C12.1, C13.1, C14.1, C15.1, LED35.P4, LED36.P4, LED37.P4, LED38.P4, LED39.P4, LED40.P4, LED41.P4, LED42.P4, LED44.P4, LED45.P4, LED46.P4, LED47.P4, LED48.P4, LED49.P4, LED50.P4, LED51.P4
- net +5V3: now also C11.1, C12.1, C13.1, C14.1, C15.1, LED35.P4, LED36.P4, LED37.P4, LED38.P4, LED39.P4, LED40.P4, LED41.P4, LED42.P4, LED44.P4, LED45.P4, LED46.P4, LED47.P4, LED48.P4, LED49.P4, LED50.P4, LED51.P4; no longer C16.1, C17.1, C18.1, C19.1, C20.1, LED52.P4, LED53.P4, LED54.P4, LED55.P4, LED56.P4, LED57.P4, LED58.P4, LED59.P4, LED61.P4, LED62.P4, LED63.P4, LED64.P4, LED65.P4, LED66.P4, LED67.P4, LED68.P4
- net +5V4: now also C16.1, C17.1, C18.1, C19.1, C20.1, LED52.P4, LED53.P4, LED54.P4, LED55.P4, LED56.P4, LED57.P4, LED58.P4, LED59.P4, LED61.P4, LED62.P4, LED63.P4, LED64.P4, LED65.P4, LED66.P4, LED67.P4, LED68.P4; no longer C21.1, C22.1, C23.1, C24.1, C25.1, LED69.P4, LED70.P4, LED71.P4, LED72.P4, LED73.P4, LED74.P4, LED75.P4, LED76.P4, LED78.P4, LED79.P4, LED80.P4, LED81.P4, LED82.P4, LED83.P4, LED84.P4, LED85.P4
- net +5V5: now also C21.1, C22.1, C23.1, C24.1, C25.1, LED69.P4, LED70.P4, LED71.P4, LED72.P4, LED73.P4, LED74.P4, LED75.P4, LED76.P4, LED78.P4, LED79.P4, LED80.P4, LED81.P4, LED82.P4, LED83.P4, LED84.P4, LED85.P4; no longer C26.1, C27.1, C28.1, C29.1, C30.1, LED100.P4, LED101.P4, LED102.P4, LED86.P4, LED87.P4, LED88.P4, LED89.P4, LED90.P4, LED91.P4, LED92.P4, LED93.P4, LED95.P4, LED96.P4, LED97.P4, LED98.P4, LED99.P4
- net +5V6: now also C26.1, C27.1, C28.1, C29.1, C30.1, LED100.P4, LED101.P4, LED102.P4, LED86.P4, LED87.P4, LED88.P4, LED89.P4, LED90.P4, LED91.P4, LED92.P4, LED93.P4, LED95.P4, LED96.P4, LED97.P4, LED98.P4, LED99.P4; no longer C31.1, C32.1, C33.1, C34.1, C35.1, LED103.P4, LED104.P4, LED105.P4, LED106.P4, LED107.P4, LED108.P4, LED109.P4, LED110.P4, LED112.P4, LED113.P4, LED114.P4, LED115.P4, LED116.P4, LED117.P4, LED118.P4, LED119.P4
- net GND1: now also C1.2, C2.2, C3.2, C4.2, C5.2, LED1.P3, LED10.P3, LED11.P3, LED12.P3, LED13.P3, LED14.P3, LED15.P3, LED16.P3, LED17.P3, LED2.P3, LED3.P3, LED4.P3, LED5.P3, LED6.P3, LED7.P3, LED8.P3, LED9.P3; no longer C10.2, C6.2, C7.2, C8.2, C9.2, LED18.P3, LED19.P3, LED20.P3, LED21.P3, LED22.P3, LED23.P3, LED24.P3, LED25.P3, LED26.P3, LED27.P3, LED28.P3, LED29.P3, LED30.P3, LED31.P3, LED32.P3, LED33.P3, LED34.P3
- net GND2: now also C10.2, C6.2, C7.2, C8.2, C9.2, LED18.P3, LED19.P3, LED20.P3, LED21.P3, LED22.P3, LED23.P3, LED24.P3, LED25.P3, LED26.P3, LED27.P3, LED28.P3, LED29.P3, LED30.P3, LED31.P3, LED32.P3, LED33.P3, LED34.P3; no longer C11.2, C12.2, C13.2, C14.2, C15.2, LED35.P3, LED36.P3, LED37.P3, LED38.P3, LED39.P3, LED40.P3, LED41.P3, LED42.P3, LED43.P3, LED44.P3, LED45.P3, LED46.P3, LED47.P3, LED48.P3, LED49.P3, LED50.P3, LED51.P3
- net GND3: now also C11.2, C12.2, C13.2, C14.2, C15.2, LED35.P3, LED36.P3, LED37.P3, LED38.P3, LED39.P3, LED40.P3, LED41.P3, LED42.P3, LED43.P3, LED44.P3, LED45.P3, LED46.P3, LED47.P3, LED48.P3, LED49.P3, LED50.P3, LED51.P3; no longer C16.2, C17.2, C18.2, C19.2, C20.2, LED52.P3, LED53.P3, LED54.P3, LED55.P3, LED56.P3, LED57.P3, LED58.P3, LED59.P3, LED60.P3, LED61.P3, LED62.P3, LED63.P3, LED64.P3, LED65.P3, LED66.P3, LED67.P3, LED68.P3
- net GND4: now also C16.2, C17.2, C18.2, C19.2, C20.2, LED52.P3, LED53.P3, LED54.P3, LED55.P3, LED56.P3, LED57.P3, LED58.P3, LED59.P3, LED60.P3, LED61.P3, LED62.P3, LED63.P3, LED64.P3, LED65.P3, LED66.P3, LED67.P3, LED68.P3; no longer C21.2, C22.2, C23.2, C24.2, C25.2, LED69.P3, LED70.P3, LED71.P3, LED72.P3, LED73.P3, LED74.P3, LED75.P3, LED76.P3, LED77.P3, LED78.P3, LED79.P3, LED80.P3, LED81.P3, LED82.P3, LED83.P3, LED84.P3, LED85.P3
- net GND5: now also C21.2, C22.2, C23.2, C24.2, C25.2, LED69.P3, LED70.P3, LED71.P3, LED72.P3, LED73.P3, LED74.P3, LED75.P3, LED76.P3, LED77.P3, LED78.P3, LED79.P3, LED80.P3, LED81.P3, LED82.P3, LED83.P3, LED84.P3, LED85.P3; no longer C26.2, C27.2, C28.2, C29.2, C30.2, LED100.P3, LED101.P3, LED102.P3, LED86.P3, LED87.P3, LED88.P3, LED89.P3, LED90.P3, LED91.P3, LED92.P3, LED93.P3, LED94.P3, LED95.P3, LED96.P3, LED97.P3, LED98.P3, LED99.P3
- net GND6: now also C26.2, C27.2, C28.2, C29.2, C30.2, LED100.P3, LED101.P3, LED102.P3, LED86.P3, LED87.P3, LED88.P3, LED89.P3, LED90.P3, LED91.P3, LED92.P3, LED93.P3, LED94.P3, LED95.P3, LED96.P3, LED97.P3, LED98.P3, LED99.P3; no longer C31.2, C32.2, C33.2, C34.2, C35.2, LED103.P3, LED104.P3, LED105.P3, LED106.P3, LED107.P3, LED108.P3, LED109.P3, LED110.P3, LED111.P3, LED112.P3, LED113.P3, LED114.P3, LED115.P3, LED116.P3, LED117.P3, LED118.P3, LED119.P3
- net LED_CK1: now also R1.1; no longer R4.1
- net LED_CK2: now also R4.1; no longer R7.1
- net LED_CK3: now also R7.1; no longer R10.1
- net LED_CK4: now also R10.1; no longer R13.1
- net LED_CK5: now also R13.1; no longer R16.1
- net LED_CK6: now also R16.1; no longer R19.1
- net LED_D1: now also R2.1; no longer R5.1
- net LED_D2: now also R5.1; no longer R8.1
- net LED_D3: now also R8.1; no longer R11.1
- net LED_D4: now also R11.1; no longer R14.1
- net LED_D5: now also R14.1; no longer R17.1
- net LED_D6: now also R17.1; no longer R20.1
- net N$1: now also LED10.P2; no longer LED2.P2
- net N$123: now also SET3.1, SET3.2; no longer SET2.1, SET2.2
- net N$164: now also SET4.1, SET4.2; no longer SET3.1, SET3.2
- net N$2: now also LED10.P1; no longer LED2.P1
- net N$205: now also SET5.1, SET5.2; no longer SET4.1, SET4.2
- net N$246: now also SET6.1, SET6.2; no longer SET5.1, SET5.2
- net N$32: now also LED9.P6; no longer MCU.1
- net N$33: now also LED9.P5; no longer MCU.3
- net N$82: now also SET2.1, SET2.2; no longer SET1.1, SET1.2
- net SW1: now also R3.1; no longer R6.1
- net SW2: now also R6.1; no longer R9.1
- net SW3: now also R9.1; no longer R12.1
- net SW4: now also R12.1; no longer R15.1
- net SW5: now also R15.1; no longer R18.1
- net SW6: now also R18.1; no longer R21.1
Routing:
- net +5V: track 149.2 -> 0.00 mm, vias 20 -> 0
- net GND: track 141.8 -> 0.00 mm, vias 18 -> 0
- net N$41: track 0.00 -> 17.4 mm, vias 0 -> 1
- net N$36 (its old number): track 17.4 -> 0.00 mm, vias 1 -> 0
- net N$287: track 17.4 -> 0.00 mm, vias 1 -> 0
- net N$280: track 16.3 -> 0.00 mm
- net LED_CK: track 13.6 -> 0.00 mm
- net SW: track 13.6 -> 0.00 mm
- net N$12: track 16.3 -> 3.42 mm
- net N$34: track 3.42 -> 16.3 mm
- net N$283: track 10.9 -> 0.00 mm
- net N$277: track 10.9 -> 0.00 mm
- net LED_D: track 9.21 -> 0.00 mm
- net N$31: track 3.42 -> 10.9 mm
- net N$5: track 10.9 -> 3.42 mm
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Other:
- board size 163 x 100 mm -> 100 x 100 mm
