File: LEDline/ledline.sch (EAGLE design)
At the start: 12 parts

Commit message: Heatsink and testpad added
Parts:
- added TP1, TP2, TP3, TP4, TP5, TP6, TP7, TP8: TPSQTP10SQ, testpad:TPSQTP10SQ
Connections:
- net GND: now also TP5.TP, TP6.TP, TP7.TP, TP8.TP
- net VCC: now also TP1.TP, TP2.TP, TP3.TP, TP4.TP
Changed lines of the file:
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@@
 <part name="D11" library="SparkFun-LED" deviceset="LED-RGB" device="PLCC-6" value="RGB"/>
 <part name="D12" library="SparkFun-LED" deviceset="LED-RGB" device="PLCC-6" value="RGB"/>
+<part name="TP2" library="testpad" deviceset="TPSQ" device="TP10SQ"/>
+<part name="TP1" library="testpad" deviceset="TPSQ" device="TP10SQ"/>
+<part name="TP3" library="testpad" deviceset="TPSQ" device="TP10SQ"/>
+<part name="TP4" library="testpad" deviceset="TPSQ" device="TP10SQ"/>
+<part name="TP5" library="testpad" deviceset="TPSQ" device="TP10SQ"/>
+<part name="TP6" library="testpad" deviceset="TPSQ" device="TP10SQ"/>
+<part name="TP7" library="testpad" deviceset="TPSQ" device="TP10SQ"/>
+<part name="TP8" library="testpad" deviceset="TPSQ" device="TP10SQ"/>
 </parts>
 <sheets>
@@
 <instance part="D11" gate="G$1" x="68.58" y="-2.54"/>
 <instance part="D12" gate="G$1" x="104.14" y="-2.54"/>
+<instance part="TP2" gate="G$1" x="-2.54" y="45.72"/>
+<instance part="TP1" gate="G$1" x="-7.62" y="45.72"/>
+<instance part="TP3" gate="G$1" x="2.54" y="45.72"/>
+<instance part="TP4" gate="G$1" x="7.62" y="45.72"/>
+<instance part="TP5" gate="G$1" x="129.54" y="43.18"/>
+<instance part="TP6" gate="G$1" x="134.62" y="43.18"/>
+<instance part="TP7" gate="G$1" x="139.7" y="43.18"/>
+<instance part="TP8" gate="G$1" x="144.78" y="43.18"/>
 </instances>
 <busses>
@@
 <net name="VCC" class="0">
 <segment>
+<pinref part="TP2" gate="G$1" pin="TP"/>
+<wire x1="-2.54" y1="48.26" x2="2.54" y2="48.26" width="0.1524" layer="91"/>
+<pinref part="TP1" gate="G$1" pin="TP"/>
+<wire x1="-7.62" y1="48.26" x2="-2.54" y2="48.26" width="0.1524" layer="91"/>
+<pinref part="TP3" gate="G$1" pin="TP"/>
+<pinref part="TP4" gate="G$1" pin="TP"/>
+<wire x1="2.54" y1="48.26" x2="7.62" y2="48.26" width="0.1524" layer="91"/>
 <pinref part="D4" gate="G$1" pin="RED-A"/>
 <pinref part="D4" gate="G$1" pin="GRN-A"/>
@@
 <wire x1="17.78" y1="50.8" x2="17.78" y2="53.34" width="0.1524" layer="91"/>
 <wire x1="17.78" y1="50.8" x2="12.7" y2="50.8" width="0.1524" layer="91"/>
-<wire x1="12.7" y1="50.8" x2="12.7" y2="33.02" width="0.1524" layer="91"/>
+<wire x1="12.7" y1="50.8" x2="12.7" y2="48.26" width="0.1524" layer="91"/>
 <pinref part="D10" gate="G$1" pin="RED-A"/>
 <pinref part="D10" gate="G$1" pin="GRN-A"/>
+<wire x1="12.7" y1="48.26" x2="12.7" y2="33.02" width="0.1524" layer="91"/>
 <wire x1="12.7" y1="33.02" x2="12.7" y2="15.24" width="0.1524" layer="91"/>
 <wire x1="12.7" y1="15.24" x2="12.7" y2="-2.54" width="0.1524" layer="91"/>
@@
 <wire x1="17.78" y1="15.24" x2="12.7" y2="15.24" width="0.1524" layer="91"/>
 <wire x1="17.78" y1="33.02" x2="12.7" y2="33.02" width="0.1524" layer="91"/>
+<wire x1="7.62" y1="48.26" x2="12.7" y2="48.26" width="0.1524" layer="91"/>
 </segment>
 </net>
@@
 <wire x1="119.38" y1="50.8" x2="119.38" y2="48.26" width="0.1524" layer="91"/>
 <wire x1="119.38" y1="50.8" x2="124.46" y2="50.8" width="0.1524" layer="91"/>
-<wire x1="124.46" y1="50.8" x2="124.46" y2="33.02" width="0.1524" layer="91"/>
+<wire x1="124.46" y1="50.8" x2="124.46" y2="45.72" width="0.1524" layer="91"/>
 <pinref part="D12" gate="G$1" pin="BLU-C"/>
 <pinref part="D12" gate="G$1" pin="GRN-C"/>
+<wire x1="124.46" y1="45.72" x2="124.46" y2="33.02" width="0.1524" layer="91"/>
 <wire x1="124.46" y1="33.02" x2="124.46" y2="15.24" width="0.1524" layer="91"/>
 <wire x1="124.46" y1="15.24" x2="124.46" y2="-2.54" width="0.1524" layer="91"/>
@@
 <wire x1="119.38" y1="15.24" x2="124.46" y2="15.24" width="0.1524" layer="91"/>
 <wire x1="119.38" y1="33.02" x2="124.46" y2="33.02" width="0.1524" layer="91"/>
-</segment>
-</net>
+<pinref part="TP8" gate="G$1" pin="TP"/>
+<pinref part="TP7" gate="G$1" pin="TP"/>
+<wire x1="144.78" y1="45.72" x2="139.7" y2="45.72" width="0.1524" layer="91"/>
+<pinref part="TP6" gate="G$1" pin="TP"/>
+<wire x1="139.7" y1="45.72" x2="134.62" y2="45.72" width="0.1524" layer="91"/>
+<pinref part="TP5" gate="G$1" pin="TP"/>
+<wire x1="134.62" y1="45.72" x2="129.54" y2="45.72" width="0.1524" layer="91"/>
+<wire x1="129.54" y1="45.72" x2="124.46" y2="45.72" width="0.1524" layer="91"/>
+</segment>
+</net>
